File: pcb/upsy-desky.kicad_sch (KiCad schematic)
At the start: 44 parts, among them J1 RJ45, J2 RJ45, J3 USB_C_ReceptacleUSB2.0, Q1 MMBT3904, Q2 MMBT3904, Q3 2N7002, Q4 2N7002, Q5 2N7002, Q6 2N7002, Q7 2N7002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

Commit message: Add test firmware and pcb changes
Parts:
- C1, C2, C5, C6: Comment (none) -> Any 5V or higher rated capacitor will work fine; MPN (none) -> GRM155R60J106ME05J; Package (none) -> 0402
- C3: Comment (none) -> Any 5V or higher rated capacitor will work fine; MPN (none) -> 0402W105K100HI; Package (none) -> 0402
- C4: Comment (none) -> Any 5V or higher rated capacitor will work fine; MPN (none) -> 0402B104K160HI; Package (none) -> 0402
- D1: MPN (none) -> 1N5817; Package (none) -> SOD-323
- D2: Comment (none) -> Any ~2.2V red LED is fine; MPN (none) -> LTST-C190KRKT; Package (none) -> 0603
- J1, J2: LCSC (none) -> C708595; MANUFACTURER Assmann WSW Components -> Amphenol ICC (FCI); MPN (none) -> 54601-708LF; Purchase https://www.digikey.com/en/products/detail/assmann-wsw-comp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 -> https://www.digikey.com/en/products/detail/amphenol-cs-fci/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
- J3: MPN (none) -> TYPE-C-31-M-12
- Q1, Q2: MPN (none) -> MMBT3904; Package (none) -> SOT-23
- Q3, Q4, Q5, Q6, Q7, Q8: MPN (none) -> 2N7002; Package (none) -> SOT-23
- R1, R2: Comment (none) -> Any 5V or higher rated resistor will work fine; MPN (none) -> RC0402JR-075R1L; Package (none) -> 0402
- R10, R11, R12, R13, R14, R15, R16, R17, R3, R4, R5, R6, R7, R8, R9: Comment (none) -> Any 5V or higher rated resistor will work fine; MPN (none) -> RC0402JR-1310KL; Package (none) -> 0402
- R18: Comment (none) -> Any 5V or higher rated resistor will work fine; MPN (none) -> RC0402JR-131KL; Package (none) -> 0402
- R19: Comment (none) -> Any 5V or higher rated resistor will work fine; MPN (none) -> RC0402FR-1322K1L; Package (none) -> 0402
- R20: Comment (none) -> Any 5V or higher rated resistor will work fine; MPN (none) -> CR0402-FX-4752GLF; Package (none) -> 0402
- R21: Comment (none) -> Any 5V or higher rated resistor will work fine; MPN (none) -> RC1005J471CS; Package (none) -> 0402
- R22: Comment (none) -> Any 5V or higher rated resistor will work fine; MPN (none) -> RMCF0402FT953R; Package (none) -> 0402
- U1: MPN (none) -> CP2102N-A02-GQFN24
- U2: MPN (none) -> AMS1117-3.3; Package (none) -> SOT-223
- U3: MPN (none) -> ESP32-WROOM-32

Commit message: misc PCB updates
Other:
- title: (none) -> Upsy Desky
Changed lines of the file:
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@@
 (kicad_sch (version 20211123) (generator eeschema)
   (paper "A4")
+  (title_block
+    (title "Upsy Desky")
+  )
   (junction (at 167.64 101.6) (diameter 0) (color 0 0 0 0)
   )
