File: pcb_v2/upsy-desky.kicad_pcb (KiCad board)
At the start: 2 copper layers, 40.9 x 58 mm, 48 parts, among them J1 RJ45, J2 RJ45, J3 USB_C_ReceptacleUSB2.0, Q1 MMBT3904, Q2 MMBT3904, Q3 BSS138, Q4 BSS138, Q5 BSS138, Q6 BSS138, Q7 BSS138, Q8 BSS138, U1 CP2102N-Axx-xQFN28, U2 AMS1117-3.3, U3 ESP32-WROOM-32

Commit message: Modify the layout
Parts:
- removed D2: LED, LED_SMD:LED_0603_1608Metric
- removed Q1, Q2: MMBT3904, Package_TO_SOT_SMD:SOT-23
- removed R22: 940, Resistor_SMD:R_0402_1005Metric
- removed REF**: MountingHole_2.2mm_M2, MountingHole:MountingHole_2.2mm_M2
- removed REF** (x2): MountingHole_3.2mm_M3, MountingHole:MountingHole_3.2mm_M3
- removed Ref**: Val**, footprints:amongy
- removed U3: ESP32-WROOM-32, RF_Module:ESP32-WROOM-32
- added C7: 15p, Capacitor_SMD:C_0402_1005Metric, F.Cu at (163.2, 80.6)
- added C8: 4.7u, Capacitor_SMD:C_0402_1005Metric, F.Cu at (149.2, 100.3)
- added C9: 100n, Capacitor_SMD:C_0402_1005Metric, F.Cu at (149.9, 104.1)
- added H1: MountingHole, MountingHole:MountingHole_2.2mm_M2_Pad, F.Cu at (130.2, 74.9)
- added H2: MountingHole, MountingHole:MountingHole_2.2mm_M2_Pad, F.Cu at (163.2, 74.9)
- added H3: MountingHole, MountingHole:MountingHole_2.2mm_M2_Pad, F.Cu at (146.7, 109.2)
- added J4: Conn_01x03_Socket, Connector:FanPinHeader_1x03_P2.54mm_Vertical, F.Cu at (129.2, 108.0)
- added J5: Screw_Terminal_01x03, TerminalBlock:TerminalBlock_Altech_AK300-3_P5.00mm, F.Cu at (160.7, 97.9)
- added J6: Conn_01x03_Pin, Connector_JST:JST_EH_B3B-EH-A_1x03_P2.50mm_Vertical, F.Cu at (162.9, 89.5)
- added SW1: SW_Push, Button_Switch_SMD:SW_Push_1P1T_NO_CK_KMR2, F.Cu at (136.5, 74.3)
- added TP1: TestPoint, TestPoint:TestPoint_Pad_D1.0mm, F.Cu at (135.3, 98.4)
- added TP10: TestPoint, TestPoint:TestPoint_Pad_D1.0mm, F.Cu at (149.9, 97.8)
- added TP11: TestPoint, TestPoint:TestPoint_Pad_D1.0mm, F.Cu at (144.8, 99.7)
- added TP2: TestPoint, TestPoint:TestPoint_Pad_D1.0mm, F.Cu at (135.3, 93.3)
- added TP3: TestPoint, TestPoint:TestPoint_Pad_D1.0mm, F.Cu at (128.3, 111.1)
- added TP4: TestPoint, TestPoint:TestPoint_Pad_D1.0mm, F.Cu at (129.5, 88.3)
- added TP5: TestPoint, TestPoint:TestPoint_Pad_D1.0mm, F.Cu at (130.8, 111.1)
- added TP6: TestPoint, TestPoint:TestPoint_Pad_D1.0mm, F.Cu at (159.4, 94.0)
- added TP7: TestPoint, TestPoint:TestPoint_Pad_D1.0mm, F.Cu at (133.3, 77.5)
- added TP8: TestPoint, TestPoint:TestPoint_Pad_D1.0mm, F.Cu at (161.9, 94.0)
- added TP9: TestPoint, TestPoint:TestPoint_Pad_D1.0mm, F.Cu at (164.5, 94.0)
- added U4: ESP32-C3-WROOM-02, PCM_Espressif:ESP32-C3-WROOM-02, F.Cu at (149.9, 84.9)
- added Y1: 32K, Crystal:Crystal_SMD_2012-2Pin_2.0x1.2mm, F.Cu at (161.3, 80.1)
- C6: value 10u -> 15p
- J1, J2: footprint footprints:ASSMANN_A-2004-2-4-LPS-N-R -> Connector_RJ:RJ45_Amphenol_54602-x08_Horizontal
- Q3, Q4, Q5, Q6, Q7, Q8: value BSS138 -> 2N7002
- R18: value 1k -> 0; moved to B.Cu
- R19: value 22.1k -> 10k
- R20: value 47.5k -> 10k
- R21: value 470 -> 0; moved to B.Cu
- R3, R4: value 10k -> 2k2
- U1: value CP2102N-Axx-xQFN28 -> VL53L0CXV0DH1; footprint Package_DFN_QFN:QFN-28-1EP_5x5mm_P0.5mm_EP3.35x3.35mm -> Sensor_Distance:ST_VL53L1x
- moved C6 33.3 mm to (163.2, 79.4), turned to 0 degrees
- moved R18 30.1 mm to (155.6, 79.4), turned to 0 degrees
- moved R21 16.2 mm to (155.6, 80.6), turned to 0 degrees
- moved C3 13.6 mm to (135.9, 78.1), turned to 180 degrees
- moved R3 11.9 mm to (148.0, 97.8), turned to -90 degrees
- moved U1 10.7 mm to (146.7, 102.9), turned to 180 degrees
- moved R19 10.2 mm to (141.6, 99.7), turned to 0 degrees
- moved R20 9.62 mm to (141.6, 98.4), turned to 0 degrees
- moved R5 8.71 mm to (135.9, 79.4), turned to 0 degrees
- moved R4 7.73 mm to (146.7, 97.8), turned to -90 degrees
- moved C5 7.73 mm to (137.8, 78.7), turned to 90 degrees
- moved C4 7.69 mm to (139.1, 78.7), turned to 90 degrees
- moved R15 6.57 mm to (156.8, 111.8)
- moved Q6 6.47 mm to (148.6, 114.3)
- moved J2 6.03 mm to (150.5, 122.3)
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Connections:
- net /GPIO16 renamed /GPIO9
- net /GPIO17 renamed /GPIO8
- net /GPIO18 renamed /GPIO7
- net /GPIO19 renamed /GPIO2
- net /GPIO21 renamed /GPIO10
- net /GPIO22 renamed /GPIO3
- C1 pad 1: +5V -> Net-(D1-K)
- C6 pad 1: +3V3 -> /GPIO0
- D1 pad 1: +5V -> Net-(D1-K)
- D1 pad 2: VBUS -> Net-(D1-A)
- J1 pad 5: +5V -> VDD
- J2 pad 5: +5V -> VDD
- J3 pad A6: /USB_D+ -> /USB_DP
- J3 pad A7: /USB_D- -> /USB_DN
- J3 pad B6: /USB_D+ -> /USB_DP
- J3 pad B7: /USB_D- -> /USB_DN
- R12 pad 2: +5V -> VDD
- R13 pad 2: +5V -> VDD
- R15 pad 2: +5V -> VDD
- R17 pad 2: +5V -> VDD
- R18 pad 1: +3V3 -> /INT
- R18 pad 2: Net-(R18-Pad2) -> /GPIO0
- R19 pad 1: VBUS -> +3V3
- R19 pad 2: Net-(R19-Pad2) -> Net-(U1-XSHUT)
- R20 pad 1: Net-(R19-Pad2) -> +3V3
- R20 pad 2: GND -> /INT
- R21 pad 1: /GPIO23 -> Net-(U1-XSHUT)
- R21 pad 2: Net-(D2-Pad2) -> /GPIO1
- R3 pad 1: /RTS -> +3V3
- R3 pad 2: Net-(Q1-Pad1) -> /SCL
- R4 pad 1: /DTR -> +3V3
- R4 pad 2: Net-(Q2-Pad1) -> /SDA
- R8 pad 2: +5V -> VDD
- R9 pad 2: +5V -> VDD
- U1 pad 1: unconnected-(U1-Pad1) -> +3V3
- U1 pad 10: unconnected-(U1-Pad10) -> /SCL
- U1 pad 11: unconnected-(U1-Pad11) -> +3V3
- U1 pad 12: unconnected-(U1-Pad12) -> GND
- U1 pad 2: unconnected-(U1-Pad2) -> GND
- U1 pad 4: /USB_D+ -> GND
- U1 pad 5: /USB_D- -> Net-(U1-XSHUT)
- U1 pad 6: +3V3 -> GND
- U1 pad 7: +3V3 -> /INT
- U1 pad 8: Net-(R19-Pad2) -> unconnected-(U1-DNC-Pad8)
- U1 pad 9: Net-(R18-Pad2) -> /SDA
- U2 pad 3: +5V -> Net-(D1-K)
Routing:
- net +5V: track 105.1 -> 0.00 mm, vias 2 -> 0
- net VDD: track 0.00 -> 85.6 mm, vias 0 -> 6
- net /LED_RGB: track 0.00 -> 42.5 mm, vias 0 -> 2
- net /USB_DP: track 0.00 -> 39.4 mm, vias 0 -> 2
- net Net-(U1-XSHUT): track 0.00 -> 37.0 mm, vias 0 -> 3
- net /INT: track 0.00 -> 35.3 mm, vias 0 -> 1
- net /USB_DN: track 0.00 -> 34.4 mm, vias 0 -> 2
- net VBUS: track 22.9 -> 57.3 mm
- net /ESP_RX: track 28.3 -> 0.00 mm, vias 2 -> 0
- net /RTS: track 28.3 -> 0.00 mm, vias 2 -> 0
- net /ESP_TX: track 26.7 -> 0.00 mm, vias 2 -> 0
- net /SCL: track 0.00 -> 26.6 mm, vias 0 -> 2
- net /GPIO23: track 26.2 -> 0.00 mm
- net /SDA: track 0.00 -> 24.8 mm
- net /GPIO0: track 30.3 -> 6.93 mm, vias 2 -> 1
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Other:
- outline, holes or cut-outs redrawn
- board text added: "1"
- board text added: "2"
- board text added: "Upsky Desky v2.0"
- board text added: "Upsy Desky by TJ Horner and Petr Hodina https://horner.tj/upsy-desky"
- board text removed: "Upsy Desky by TJ Horner https://horner.tj/upsy-desky"

Commit message: Several improvements:
- Improved GND connection to the ESP32 module.
- Connected the UART signals to SBU pins.
- Rounded corners
Connections:
- H1 pad 1: GND -> (no net)
- H2 pad 1: GND -> (no net)
- H3 pad 1: GND -> (no net)
- J3 pad A8: unconnected-(J3-SBU1-PadA8) -> /DBG_RX
- J3 pad B8: unconnected-(J3-SBU2-PadB8) -> /DBG_TX
- Q3 pad 2: /GPIO7 -> /GPIO9
- Q4 pad 2: /GPIO9 -> /GPIO7
- R6 pad 1: /GPIO7 -> /GPIO9
- R7 pad 1: /GPIO9 -> /GPIO7
Routing:
- net /DBG_RX: track 9.18 -> 48.2 mm, vias 0 -> 2
- net /DBG_TX: track 12.3 -> 50.1 mm, vias 0 -> 2
- net VBUS: track 57.3 -> 60.0 mm
- net /GPIO7: track 31.0 -> 32.6 mm
- net /GPIO8: track 28.5 -> 29.8 mm
- net /INT: track 35.3 -> 36.4 mm
- net /GPIO9: track 28.0 -> 28.9 mm
- net Net-(U1-XSHUT): track 37.0 -> 37.8 mm
Other:
- outline, holes or cut-outs redrawn
